File: pcb/corne choc.kicad_pcb (KiCad board)
At the start: 2 copper layers, 265.7 x 87.7 mm, 168 parts, among them J1 MJ-4PP-9, J2 OLED, J3 MJ-4PP-9, J4 OLED, SW1 SW_PUSH, SW10 SW_PUSH, SW11 SW_PUSH, SW12 SW_PUSH, SW13 SW_PUSH, SW14 SW_PUSH, SW15 SW_PUSH, SW16 SW_PUSH, SW17 SW_PUSH, SW18 SW_PUSH, SW19 SW_PUSH, SW2 SW_PUSH, SW20 SW_PUSH, SW21 SW_PUSH, SW22 SW_PUSH, SW23 SW_PUSH, SW24 SW_PUSH, SW25 SW_PUSH, SW26 SW_PUSH, SW27 SW_PUSH, SW28 SW_PUSH, SW29 SW_PUSH, SW3 SW_PUSH, SW30 SW_PUSH, SW31 SW_PUSH, SW32 SW_PUSH, SW33 SW_PUSH, SW34 SW_PUSH, SW35 SW_PUSH, SW36 SW_PUSH, SW37 SW_PUSH, SW38 SW_PUSH, SW39 SW_PUSH, SW4 SW_PUSH, SW40 SW_PUSH, SW41 SW_PUSH, SW42 SW_PUSH, SW5 SW_PUSH, SW6 SW_PUSH, SW7 SW_PUSH, SW8 SW_PUSH, SW9 SW_PUSH, U1 ProMicro, U2 ProMicro

Commit message: Right-thumb trackpoint: widen inner edges, jacks to top edge, module header TP1
Generated by tools/build.sh from the upstream board. SW42, D42 and the right
OLED header are removed; TP1 (Pro Micro pattern, pins 5/6/21/23 wired to
GP2/GP3/3V3/GND) takes the thumb spot. Both halves widen 6.2 mm on the inner
edge so the TRRS jacks face the top edge beside the controllers. DRC matches
upstream apart from pre-existing LED cutout warnings.
Parts:
- removed D42: D, kbd:D3_SMD_v2
- removed J4: OLED, holykeebs:OLED_1side_1mm_holes
- removed SW42: SW_PUSH, holykeebs:SW_choc_v1_HS_CPG135001S30_1.5u
- added TP1: holykeebs trackpoint module, holykeebs:ProMicro_1mm_holes, F.Cu at (176.3, 123.0)
- moved J3 48.4 mm to (162.3, 57.2), turned to 0 degrees
- moved J1 47.6 mm to (149.4, 57.2), turned to 0 degrees
- moved D22 12.4 mm to (278.7, 64.4)
- moved D29 12.4 mm to (260.7, 79.5)
- moved D35 12.4 mm to (260.0, 98.3)
- moved LED28 12.4 mm to (276.4, 73.8)
- moved LED31 12.4 mm to (276.2, 90.9)
- moved ? 12.4 mm to (204.5, 72.0)
- moved D25 12.4 mm to (224.5, 56.6)
- moved D26 12.4 mm to (206.9, 59.5)
- moved D27 12.4 mm to (188.2, 60.9)
- moved D30 12.4 mm to (242.6, 75.7)
- moved D31 12.4 mm to (224.9, 73.2)
- moved D32 12.4 mm to (207.1, 76.4)
- moved D33 12.4 mm to (188.6, 77.8)
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Routing:
- net data_r: track 62.1 -> 19.0 mm
- net data: track 45.0 -> 8.02 mm
- net col5_r: track 107.9 -> 71.7 mm
- net VCC: track 65.9 -> 97.4 mm, vias 0 -> 2
- net SCL_r: track 24.0 -> 46.2 mm, vias 0 -> 2
- net SDA_r: track 27.6 -> 46.8 mm, vias 0 -> 2
- net row3_r: track 83.0 -> 64.7 mm
- net VDD: track 87.8 -> 104.3 mm, vias 2 -> 3
- net GNDA: track 554.6 -> 538.6 mm
- net Net-(D42-A): track 7.03 -> 0.00 mm
Other:
- board size 265.7 x 87.7 mm -> 278.1 x 90.4 mm

Commit message: Trackpoint at the right outer thumb key with an SK8707-01 sensor and driver
Replaces the earlier holykeebs-module design. The board is stock except at
SW40: switch, diode and hidden LED removed (RGB chain bridged), sensor on the
front at the key centre, driver on the back beneath it, PS/2 to U2 pins 11/12
(GP8/GP9). Routing uses a small grid router; DRC matches upstream apart from
pre-existing LED-cutout warnings.
Parts:
- removed D40: D, kbd:D3_SMD_v2
- removed LED52: YS-SK6812MINI-E, PCM_marbastlib-various:LED_6028R
- removed SW40: SW_PUSH, holykeebs:SW_choc_v1_HS_CPG135001S30_1u
- added D42: D, kbd:D3_SMD_v2, B.Cu at (165.7, 113.9)
- added J4: OLED, holykeebs:OLED_1side_1mm_holes, F.Cu at (158.5, 94.0)
- added SW42: SW_PUSH, holykeebs:SW_choc_v1_HS_CPG135001S30_1.5u, B.Cu at (166.1, 123.3)
- added TP2: SK8707-01 driver, SK8707-01_driver, B.Cu at (206.7, 116.3)
- TP1: value holykeebs trackpoint module -> SK8707-01 sensor; footprint holykeebs:ProMicro_1mm_holes -> SK8707-01_sensor
- moved J3 48.4 mm to (152.8, 104.7), turned to 90 degrees
- moved J1 47.6 mm to (146.6, 104.7), turned to -90 degrees
- moved TP1 30.9 mm to (206.7, 117.5), turned to 180 degrees
- moved D22 12.4 mm to (266.3, 64.4)
- moved D29 12.4 mm to (248.3, 79.5)
- moved D35 12.4 mm to (247.6, 98.3)
- moved LED28 12.4 mm to (264.0, 73.8)
- moved LED31 12.4 mm to (263.8, 90.9)
- moved ? 12.4 mm to (192.1, 72.0)
- moved D25 12.4 mm to (212.1, 56.6)
- moved D26 12.4 mm to (194.5, 59.5)
- moved D27 12.4 mm to (175.8, 60.9)
- moved D30 12.4 mm to (230.2, 75.7)
- moved D31 12.4 mm to (212.5, 73.2)
- moved D32 12.4 mm to (194.7, 76.4)
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Connections:
- LED49 pad 4: Net-(LED49-DIN) -> Net-(LED52-DIN)
- U2 pad 11: unconnected-(U2-8/B4-Pad11) -> TP_DATA
- U2 pad 12: unconnected-(U2-9/B5-Pad12) -> TP_CLK
Routing:
- net TP_DATA: track 0.00 -> 69.3 mm, vias 0 -> 3
- net TP_CLK: track 0.00 -> 65.9 mm, vias 0 -> 4
- net GNDA: track 538.6 -> 584.4 mm, vias 2 -> 4
- net data_r: track 19.0 -> 62.1 mm
- net VDD: track 104.3 -> 145.4 mm, vias 3 -> 5
- net data: track 8.02 -> 45.0 mm
- net col5_r: track 71.7 -> 107.9 mm
- net VCC: track 97.4 -> 65.9 mm, vias 2 -> 0
- net col3_r: track 155.4 -> 126.4 mm
- net Net-(LED49-DIN): track 26.2 -> 0.00 mm, vias 2 -> 0
- net Net-(LED52-DIN): track 14.4 -> 40.1 mm, vias 2 -> 4
- net SCL_r: track 46.2 -> 24.0 mm, vias 2 -> 0
- net SDA_r: track 46.8 -> 27.6 mm, vias 2 -> 0
- net Net-(D44-K): track 548.4 -> 555.7 mm
- net Net-(D42-A): track 0.00 -> 7.03 mm
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Other:
- board size 278.1 x 90.4 mm -> 265.7 x 87.7 mm
