File: pcb/corne choc.kicad_pcb (KiCad board)
At the start: 2 copper layers, 278.1 x 88.4 mm, 167 parts, among them J1 MJ-4PP-9, J2 OLED, J3 MJ-4PP-9, J4 OLED, SW1 SW_PUSH, SW10 SW_PUSH, SW11 SW_PUSH, SW12 SW_PUSH, SW13 SW_PUSH, SW14 SW_PUSH, SW15 SW_PUSH, SW16 SW_PUSH, SW17 SW_PUSH, SW18 SW_PUSH, SW19 SW_PUSH, SW2 SW_PUSH, SW20 SW_PUSH, SW21 SW_PUSH, SW22 SW_PUSH, SW23 SW_PUSH, SW24 SW_PUSH, SW25 SW_PUSH, SW26 SW_PUSH, SW27 SW_PUSH, SW28 SW_PUSH, SW29 SW_PUSH, SW3 SW_PUSH, SW30 SW_PUSH, SW31 SW_PUSH, SW32 SW_PUSH, SW33 SW_PUSH, SW34 SW_PUSH, SW35 SW_PUSH, SW36 SW_PUSH, SW37 SW_PUSH, SW38 SW_PUSH, SW39 SW_PUSH, SW4 SW_PUSH, SW41 SW_PUSH, SW42 SW_PUSH, SW43 SW_PUSH, SW44 SW_PUSH, SW5 SW_PUSH, SW6 SW_PUSH, SW7 SW_PUSH, SW8 SW_PUSH, SW9 SW_PUSH, U1 ProMicro, U2 ProMicro

Commit message: v2.1: 1.15 mm key-to-edge gap, matching switch orientation, LED moves
- Keycaps sit 1.15 mm from the edge wherever it follows them; outer side
  edges move out, and every hot-swap socket pad clears the edge by 0.33 mm.
- The left inner thumb keys no longer turn 180 degrees: every switch, and
  every per-key LED, faces the same way.
- Underglow LED32 and its left twin LED5 move, mirrored, clear of the
  trackpoint driver's hand-soldered pads.
- Mounting holes for the unused OLED cover removed (tools/strip.py).
- Plates follow the moved outer edges; renders show both plates fitted.
- Build: finish pass runs until no dangling copper is left.
Parts:
- removed the h2 at (181.2, 102.3)
- removed the h2 at (130.5, 102.3)
- removed the h2 at (150.6, 106.0)
- removed the h2 at (161.2, 106.0)
- moved D21 18.3 mm to (127.2, 119.6), turned to 75 degrees
- moved D45 18.3 mm to (135.7, 104.9), turned to 75 degrees
- moved LED5 13.6 mm to (72.2, 104.6)
- moved LED32 13.6 mm to (239.5, 104.6)
- moved LED55 9.40 mm to (137.5, 117.1), turned to -30 degrees
- moved LED27 9.40 mm to (129.0, 131.9), turned to -30 degrees
- turned SW21 to -30 degrees
- turned SW43 to -30 degrees
Routing:
- net GNDA: track 515.4 -> 484.3 mm
- net row3: track 115.1 -> 89.8 mm, vias 3 -> 5
- net Net-(LED31-DOUT): track 63.3 -> 45.8 mm
- net GND: track 574.6 -> 592.1 mm, vias 14 -> 12
- net Net-(LED32-DOUT): track 45.6 -> 59.6 mm
- net Net-(LED4-DOUT): track 51.2 -> 37.8 mm
- net Net-(LED51-DIN): track 36.6 -> 26.6 mm, vias 2 -> 4
- net Net-(D44-K): track 544.7 -> 535.6 mm, vias 13 -> 9
- net Net-(D45-A): track 10.3 -> 3.68 mm
- net Net-(D21-A): track 3.70 -> 10.2 mm
- net Net-(LED24-DIN): track 20.7 -> 27.1 mm
- net Net-(LED5-DOUT): track 44.2 -> 49.7 mm
- net Net-(LED33-DOUT): track 32.9 -> 27.6 mm
- net col2: track 159.3 -> 164.3 mm, vias 3 -> 2
- net Net-(LED27-DOUT): track 19.5 -> 21.7 mm, vias 2 -> 0
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Other:
- board size 278.1 x 88.4 mm -> 278.5 x 88.6 mm

Commit message: v2.1: driver pads per drawing, diagonal plate edge, no-OLED renders
- Trackpoint driver host pads follow Sprintek's drawing: 1.0 mm wide at
  1.80 mm pitch, leaving 0.8 mm between them for hand soldering.
- The switch plate carries the upper inner thumb key's top edge straight
  on to its inner edge (2.6 mm clear of the OLED header) instead of a step.
- Render script gains assembled top-down and no-OLED views.
Routing:
- net Net-(LED54-DOUT): track 19.5 -> 25.9 mm
- net col5_r: track 105.8 -> 100.3 mm, vias 3 -> 5
- net GND: track 592.1 -> 597.4 mm
- net row3_r: track 88.0 -> 84.6 mm, vias 2 -> 4
- net Net-(D44-K): track 535.6 -> 538.2 mm, vias 9 -> 8
- net Net-(LED51-DIN): track 26.6 -> 28.0 mm
- net GNDA: track 484.3 -> 482.9 mm
- net Net-(LED33-DOUT): track 27.6 -> 26.9 mm
