File: pcb/corne choc plate.kicad_pcb (KiCad board)
At the start: 2 copper layers, 130 x 87.7 mm, 28 parts, among them SW1 SW_PUSH, SW10 SW_PUSH, SW11 SW_PUSH, SW12 SW_PUSH, SW13 SW_PUSH, SW14 SW_PUSH, SW15 SW_PUSH, SW16 SW_PUSH, SW17 SW_PUSH, SW18 SW_PUSH, SW19 SW_PUSH, SW2 SW_PUSH, SW20 SW_PUSH, SW21 SW_PUSH, SW3 SW_PUSH, SW4 SW_PUSH, SW5 SW_PUSH, SW6 SW_PUSH, SW7 SW_PUSH, SW8 SW_PUSH, SW9 SW_PUSH

Commit message: v2: wider inner edges, jacks at the top, split inner thumb keys, peaked top edges
Both halves widen 6.2 mm inward with the TRRS jacks facing the top edge; each
inner 1.5u thumb becomes two 1u keys at the same angle (new key on col2, with
diode and LED in the chain); edges sit 0.95 mm from the inner thumb keycaps;
top edges peak at the middle-finger column. New switch plate and FR4 bottom.
Routing is DRC-driven (autoconnect + maze); DRC matches upstream apart from
warnings.
Parts:
- removed SW21: SW_PUSH, kbd:SW_Hole
- added SW45: SW_PUSH, kbd:SW_Hole, F.Cu at (164.3, 127.2)
- added SW46: SW_PUSH, kbd:SW_Hole, F.Cu at (155.3, 111.6)
Other:
- board size 130 x 87.7 mm -> 136.2 x 88.2 mm
