File: pcb/bottom.kicad_pcb (KiCad board)
At the start: 2 copper layers, 278.1 x 88.2 mm, 10 parts

Commit message: v2.1: thumb arc, key-following edges, roomier trackpoint
- Thumb keys on one arc on both halves (0/15/30 degrees); the split inner
  keys turn like the others and stack one row apart (tools/thumbs.py).
- Edge round the thumbs redrawn from the keys: 0.95 mm from the inner
  keycaps, one level line under the middle and outer keys, and a 60-degree
  outer slant cornered off the trackpoint sensor. Halves identical.
- Trackpoint stem 3.4 mm lower in the same board footprint.
- Holykeebs and Corne logos removed.
- Separate right switch plate with an opening for the sensor.
- Router stops on the copper it is joining; ground islands are joined to
  the main ground; sensor links routed like other nets.
- Renders use KLP Lame keycaps; tools/demo.sh rebuilds them.
Other:
- board size 278.1 x 88.2 mm -> 278.1 x 88.4 mm

Commit message: v2.1: 1.15 mm key-to-edge gap, matching switch orientation, LED moves
- Keycaps sit 1.15 mm from the edge wherever it follows them; outer side
  edges move out, and every hot-swap socket pad clears the edge by 0.33 mm.
- The left inner thumb keys no longer turn 180 degrees: every switch, and
  every per-key LED, faces the same way.
- Underglow LED32 and its left twin LED5 move, mirrored, clear of the
  trackpoint driver's hand-soldered pads.
- Mounting holes for the unused OLED cover removed (tools/strip.py).
- Plates follow the moved outer edges; renders show both plates fitted.
- Build: finish pass runs until no dangling copper is left.
Other:
- board size 278.1 x 88.4 mm -> 278.5 x 88.6 mm
