File: pcb/dual/corne choc dual.kicad_pcb (KiCad board)
At the start: 2 copper layers, 278.5 x 88.6 mm, 163 parts, among them J1 MJ-4PP-9, J2 OLED, J3 MJ-4PP-9, J4 OLED, SW1 SW_PUSH, SW10 SW_PUSH, SW11 SW_PUSH, SW12 SW_PUSH, SW13 SW_PUSH, SW14 SW_PUSH, SW15 SW_PUSH, SW16 SW_PUSH, SW17 SW_PUSH, SW18 SW_PUSH, SW19 SW_PUSH, SW2 SW_PUSH, SW20 SW_PUSH, SW21 SW_PUSH, SW22 SW_PUSH, SW23 SW_PUSH, SW24 SW_PUSH, SW25 SW_PUSH, SW26 SW_PUSH, SW27 SW_PUSH, SW28 SW_PUSH, SW29 SW_PUSH, SW3 SW_PUSH, SW30 SW_PUSH, SW31 SW_PUSH, SW32 SW_PUSH, SW33 SW_PUSH, SW34 SW_PUSH, SW35 SW_PUSH, SW36 SW_PUSH, SW37 SW_PUSH, SW38 SW_PUSH, SW39 SW_PUSH, SW4 SW_PUSH, SW41 SW_PUSH, SW42 SW_PUSH, SW43 SW_PUSH, SW44 SW_PUSH, SW5 SW_PUSH, SW6 SW_PUSH, SW7 SW_PUSH, SW8 SW_PUSH, SW9 SW_PUSH, U1 ProMicro, U2 ProMicro

Commit message: Dual-trackpoint variant (build.sh dual) alongside the single
- tools/outer_thumb.py places a trackpoint on either half (one half per run);
  the dual build puts one on each outer thumb key, into pcb/dual/ and
  fab/dual/, with one switch-plate design (sensor opening) for both halves.
- Left trackpoint: same pins (GP8/GP9) and 3.3 V source as the right.
- Router keeps 0.3 mm from other copper (diagonals had cut inside 0.2 mm);
  each driver's ground pin joins by track, not by the pour.
- fab.sh and demo renders handle either variant; the 1.111x printout is
  gone (print with scaling off instead).
Parts:
- removed D19: D, kbd:D3_SMD_v2
- removed LED25: YS-SK6812MINI-E, PCM_marbastlib-various:LED_6028R
- removed SW19: SW_PUSH, holykeebs:SW_choc_v1_HS_CPG135001S30_1u
- added TP3: SK8707-01 sensor, SK8707-01_sensor, F.Cu at (92.6, 120.9)
- added TP4: SK8707-01 driver, SK8707-01_driver, B.Cu at (92.6, 116.1)
Connections:
- LED22 pad 4: Net-(LED22-DIN) -> Net-(LED25-DIN)
- U1 pad 11: unconnected-(U1-8/B4-Pad11) -> TP_DATA_L
- U1 pad 12: unconnected-(U1-9/B5-Pad12) -> TP_CLK_L
Routing:
- net TP_CLK_L: track 0.00 -> 69.3 mm, vias 0 -> 1
- net TP_DATA_L: track 0.00 -> 66.7 mm, vias 0 -> 1
- net VCC: track 83.9 -> 150.1 mm, vias 2 -> 3
- net col3: track 124.6 -> 97.3 mm
- net Net-(LED22-DIN): track 26.6 -> 0.00 mm, vias 2 -> 0
- net Net-(D43-K): track 522.4 -> 506.0 mm, vias 6 -> 8
- net row3: track 89.9 -> 77.7 mm, vias 5 -> 7
- net Net-(D44-K): track 545.7 -> 535.3 mm
- net Net-(D21-A): track 10.2 -> 3.68 mm
- net Net-(D19-A): track 5.24 -> 0.00 mm
- net Net-(LED25-DIN): track 38.4 -> 43.0 mm, vias 2 -> 4
- net Net-(LED24-DIN): track 27.1 -> 30.8 mm, vias 2 -> 4
- net Net-(LED27-DIN): track 21.9 -> 24.1 mm
- net GND: track 593.4 -> 595.0 mm, vias 12 -> 20
- net row3_r: track 88.6 -> 89.9 mm
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
Commit message: Thumb cluster on the index-aligned arc, wider inner edge, 15-degree marks
- The thumb cluster sits 1.37 mm further in and 0.98 mm higher, so the middle
  thumb key meets the bottom index key the way it meets the inner key (same
  corner gap, opening at 15 degrees); the trackpoint moves with it.
- The inner straight edge moves out by what the upper inner thumb key needs
  to keep the 1.15 mm gap (6.92 mm in all); jacks stay centred in the strip,
  1.24 mm from the controller pins.
- Silkscreen protractor marks ("15°") in the three thumb gaps, on the PCB
  front and both faces of every switch plate.
- Both variants rebuilt; plate renders include silkscreen.
Parts:
- moved D42 11.1 mm to (170.2, 126.4)
- moved D21 1.69 mm to (128.6, 118.7)
- moved D45 1.69 mm to (137.1, 103.9)
- moved LED55 1.69 mm to (138.9, 116.2)
- moved LED26 1.69 mm to (112.8, 123.7)
- moved D20 1.69 mm to (107.9, 112.3)
- moved SW20 1.69 mm to (114.0, 119.1)
- moved LED27 1.69 mm to (130.4, 130.9)
- moved SW21 1.69 mm to (132.7, 126.8)
- moved SW43 1.69 mm to (141.2, 112.1)
- moved D46 1.69 mm to (161.7, 111.6)
- moved D41 1.69 mm to (189.3, 116.4)
- moved LED53 1.69 mm to (198.9, 123.7)
- moved SW42 1.69 mm to (179.0, 126.8)
- moved SW44 1.69 mm to (170.5, 112.1)
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Routing:
- net GNDA: track 555.7 -> 501.6 mm, vias 8 -> 9
- net GND: track 595.0 -> 570.6 mm, vias 20 -> 18
- net Net-(LED52-DIN): track 55.8 -> 39.9 mm
- net Net-(LED32-DOUT): track 61.9 -> 77.4 mm, vias 6 -> 4
- net data_r: track 32.7 -> 19.4 mm, vias 1 -> 0
- net TP_DATA: track 77.3 -> 66.2 mm, vias 2 -> 3
- net row3_r: track 89.9 -> 79.3 mm, vias 2 -> 5
- net Net-(LED50-DOUT): track 36.0 -> 45.4 mm, vias 2 -> 6
- net Net-(LED25-DIN): track 43.0 -> 50.4 mm
- net Net-(D42-A): track 9.76 -> 2.54 mm
- net Net-(LED33-DOUT): track 32.9 -> 27.7 mm
- net TP_DATA_L: track 66.7 -> 62.7 mm
- net Net-(LED27-DIN): track 24.1 -> 20.5 mm, vias 0 -> 2
- net row3: track 77.7 -> 80.6 mm, vias 7 -> 5
- net Net-(LED24-DIN): track 30.8 -> 28.2 mm
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Other:
- board size 278.5 x 88.6 mm -> 278.5 x 87.6 mm
- board text added: "15°"
