File: pcb/dual/bottom.kicad_pcb (KiCad board)
At the start: 2 copper layers, 278.5 x 88.6 mm, 10 parts

Commit message: Thumb cluster on the index-aligned arc, wider inner edge, 15-degree marks
- The thumb cluster sits 1.37 mm further in and 0.98 mm higher, so the middle
  thumb key meets the bottom index key the way it meets the inner key (same
  corner gap, opening at 15 degrees); the trackpoint moves with it.
- The inner straight edge moves out by what the upper inner thumb key needs
  to keep the 1.15 mm gap (6.92 mm in all); jacks stay centred in the strip,
  1.24 mm from the controller pins.
- Silkscreen protractor marks ("15°") in the three thumb gaps, on the PCB
  front and both faces of every switch plate.
- Both variants rebuilt; plate renders include silkscreen.
Other:
- board size 278.5 x 88.6 mm -> 278.5 x 87.6 mm

Commit message: Petrock-41/40: rebuild from the stock Corne Choc with minimal copper change
Parts move to the final layout dragging their copper, crowded copper is
nudged inside the new edge, only copper off the board or in a clash the
stock board didn't have is cut, and only what is then open is routed,
never ripping up stock copper. About 60% of the stock copper stays.

Lighting is dropped for this build (no_leds.py). The pinky and ring
fourth keys join the column wire they land on (row 3); the upper inner
thumb takes col 0. The trackpoint reset line, LED power switch,
underglow grid and 15-degree marks are gone, with the old rip-up and
prune steps. Boards renamed: petrock-41 (single), petrock-40 (dual).
Parts:
- removed H10, H9: , 
- moved H3 170.7 mm to (204.5, 72.0)
- moved H7 130.5 mm to (231.8, 111.2)
- moved H8 92.0 mm to (186.0, 113.7)
- moved H4 89.1 mm to (125.7, 113.7)
- moved H6 56.1 mm to (246.2, 126.0)
- moved H1 55.1 mm to (79.9, 111.2)
- moved H5 45.6 mm to (107.3, 72.0)
- moved H2 20.0 mm to (65.5, 126.0)
Other:
- board size 278.5 x 87.6 mm -> 242.5 x 87.9 mm
