File: pcb/none/petrock-42 plate.kicad_pcb (KiCad board)
At the start: 2 copper layers, 119.3 x 87.9 mm, 25 parts, among them SW1 SW_PUSH, SW10 SW_PUSH, SW11 SW_PUSH, SW12 SW_PUSH, SW13 SW_PUSH, SW14 SW_PUSH, SW15 SW_PUSH, SW16 SW_PUSH, SW17 SW_PUSH, SW18 SW_PUSH, SW19 SW_PUSH, SW2 SW_PUSH, SW20 SW_PUSH, SW3 SW_PUSH, SW4 SW_PUSH, SW5 SW_PUSH, SW6 SW_PUSH, SW7 SW_PUSH, SW8 SW_PUSH, SW9 SW_PUSH

Commit message: Boards, plates and renders built from 86592b8 (the hash printed on the boards); adds the Petrock-42
Parts:
- added SW21: SW_PUSH, kbd:SW_Hole, F.Cu at (250.8, 99.9)
- moved SW10 56.9 mm to (201.1, 116.4)
- moved SW14 51.0 mm to (232.8, 114.6)
- moved SW18 51.0 mm to (250.8, 116.9)
- moved SW13 26.4 mm to (214.8, 95.2)
- moved SW17 26.4 mm to (232.8, 97.6)
- moved SW19 17.0 mm to (250.8, 65.9)
- moved SW15 17.0 mm to (232.8, 63.6)
- moved SW11 17.0 mm to (214.8, 61.2)
- moved SW12 17.0 mm to (214.8, 78.2)
- moved SW16 17.0 mm to (232.8, 80.6)
- moved SW20 17.0 mm to (250.8, 82.9)
Other:
- outline, holes or cut-outs redrawn
