File: pcb/none/petrock-42.kicad_pcb (KiCad board)
At the start: 2 copper layers, 242.5 x 87.9 mm, 102 parts, among them J1 MJ-4PP-9, J2 OLED, J3 MJ-4PP-9, J4 OLED, SW1 SW_PUSH, SW10 SW_PUSH, SW11 SW_PUSH, SW12 SW_PUSH, SW13 SW_PUSH, SW14 SW_PUSH, SW15 SW_PUSH, SW16 SW_PUSH, SW17 SW_PUSH, SW18 SW_PUSH, SW19 SW_PUSH, SW2 SW_PUSH, SW20 SW_PUSH, SW21 SW_PUSH, SW22 SW_PUSH, SW23 SW_PUSH, SW24 SW_PUSH, SW25 SW_PUSH, SW26 SW_PUSH, SW27 SW_PUSH, SW29 SW_PUSH, SW3 SW_PUSH, SW30 SW_PUSH, SW31 SW_PUSH, SW32 SW_PUSH, SW33 SW_PUSH, SW34 SW_PUSH, SW35 SW_PUSH, SW36 SW_PUSH, SW37 SW_PUSH, SW38 SW_PUSH, SW39 SW_PUSH, SW4 SW_PUSH, SW41 SW_PUSH, SW42 SW_PUSH, SW43 SW_PUSH, SW44 SW_PUSH, SW5 SW_PUSH, SW6 SW_PUSH, SW8 SW_PUSH, SW9 SW_PUSH, U1 ProMicro, U2 ProMicro

Commit message: Boards, plates and renders built from 86592b8 (the hash printed on the boards); adds the Petrock-42
Parts:
- removed A1: SK8707-01 sensor, SK8707-01_sensor
- removed A2: SK8707-01 driver, SK8707-01_driver
- added D40: D, kbd:D3_SMD_v2, B.Cu at (210.9, 112.7)
- added SW40: SW_PUSH, holykeebs:SW_choc_v1_HS_CPG135001S30_1u, B.Cu at (217.5, 116.4)
Connections:
- SW41 pad 1: col3_r -> col4_r
- SW42 pad 1: col4_r -> col5_r
- SW44 pad 1: col5_r -> col0_r
- U2 pad 1: TP_CLK -> (no net)
- U2 pad 2: TP_DATA -> (no net)
Routing:
- net VDD: track 201.0 -> 55.5 mm, vias 1 -> 0
- net TP_DATA: track 127.7 -> 0.00 mm, vias 1 -> 0
- net TP_CLK: track 124.7 -> 0.00 mm, vias 1 -> 0
- net col3_r: track 209.7 -> 152.6 mm
- net col0_r: track 0.00 -> 44.0 mm
- net TP_S4: track 29.8 -> 0.00 mm, vias 1 -> 0
- net TP_S3: track 26.6 -> 0.00 mm, vias 1 -> 0
- net TP_S2: track 23.4 -> 0.00 mm, vias 1 -> 0
- net col4_r: track 161.0 -> 137.9 mm
- net TP_S1: track 20.2 -> 0.00 mm, vias 1 -> 0
- net row3_r: track 173.6 -> 178.5 mm
- net col5_r: track 113.9 -> 117.3 mm
- net Net-(D40-A): track 0.00 -> 3.36 mm
- net GNDA: track 4.31 -> 2.50 mm, vias 107 -> 132
